Commit message: Gemelo digital funcional

File: src/kia_gd/urdf/ur5.urdf (robot description, URDF)
Before this commit: robot UR5, 7 links, 6 joints
Joints:
- joint J1_J2: axis 1 0 0 -> -1 0 0; origin xyz=0 0.0 0.79 rpy=0 0 3.141592 -> xyz=0 0.0 0.79 rpy=-1.57 0 3.141592
- joint J3_J4: axis 1 0 0 -> -1 0 0; origin xyz=0 0.01 3.95 rpy=0 0 3.141592 -> xyz=0 0.01 3.95 rpy=-1.57 0 3.141592

Commit message: .

File: src/kia_gd/urdf/ur5.urdf (robot description, URDF)
Before this commit: robot UR5, 7 links, 6 joints
Joints:
- joint J4_J5: origin xyz=-1.22 0 0 rpy=0 0 3.141592 -> xyz=-1.22 0 0 rpy=0 0 0

Commit message: .

File: src/kia_gd/urdf/ur5.urdf (robot description, URDF)
Before this commit: robot UR5, 7 links, 6 joints
Links:
- link Base: geometry visual mesh filename=package://kia_gd/meshes/Base_scaled.stl scale=1 1 1
- link J1: geometry visual mesh filename=package://kia_gd/meshes/J1_scaled.stl scale=1 1 1
- link J2: geometry visual mesh filename=package://kia_gd/meshes/J2_scaled.stl scale=1 1 1
- link J3: geometry visual mesh filename=package://kia_gd/meshes/J3.stl scale=0.001 0.001 0.001
- link J4: geometry visual mesh filename=package://kia_gd/meshes/J4_scaled.stl scale=1 1 1
- link J5: geometry visual mesh filename=package://kia_gd/meshes/J5_scaled.stl scale=1 1 1
- link J6: geometry visual mesh filename=package://kia_gd/meshes/J6_scaled.stl scale=1 1 1
Joints:
- joint Base_J1: origin xyz=0 0.0 0.0 rpy=0 0 0 -> xyz=0.5 0.0 0.0 rpy=0 0 0
- joint J1_J2: origin xyz=0 0.0 0.79 rpy=-1.57 0 3.141592 -> xyz=0 0.00 0.090 rpy=-1.57 0 3.141592
- joint J2_J3: origin xyz=0 -0.02 4.28 rpy=0 0 3.141592 -> xyz=0 0.00 0.430 rpy=0 0 3.141592
- joint J3_J4: origin xyz=0 0.01 3.95 rpy=-1.57 0 3.141592 -> xyz=0 0.001 0.393 rpy=-1.57 0 3.141592
- joint J4_J5: origin xyz=-1.22 0 0 rpy=0 0 0 -> xyz=-0.117 0 0 rpy=0 0 0
- joint J5_J6: origin xyz=0 -0.02 0.97 rpy=0 0 3.141592 -> xyz=0 0 0.097 rpy=0 0 3.141592
